File: KiCAD/YM2151.sch (KiCad schematic (older format))
At the start: 37 parts, among them J1 Audio-Jack-3_2Switches, P1 Power, P2 Analog, P3 Digital, P4 Digital, P5 CONN_01X01, P6 CONN_01X01, P7 CONN_01X01, P8 CONN_01X01, Q1 2SC1815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

Commit message: 部品表整備
Parts:
- O1: value OSCILLATOR -> 3.579545MHz
- U4: value 74LS138 -> 74HC138
Changed lines of the file:
@@
 P 1400 7150
 F 0 "O1" H 1200 7450 60  0000 C CNN
-F 1 "OSCILLATOR" H 1500 6850 60  0000 C CNN
+F 1 "3.579545MHz" H 1500 6850 60  0000 C CNN
 F 2 "Oscillator:Oscillator_DIP-14" H 1400 7150 60  0001 C CNN
 F 3 "" H 1400 7150 60  0001 C CNN
@@
 P 5500 1650
 F 0 "U4" H 5250 2100 50  0000 C CNN
-F 1 "74LS138" H 5750 2100 50  0000 C CNN
+F 1 "74HC138" H 5750 2100 50  0000 C CNN
 F 2 "Package_DIP:DIP-16_W7.62mm_Socket" H 5500 1650 50  0001 C CNN
 F 3 "http://www.ti.com/lit/gpn/sn74LS138" H 5500 1650 50  0001 C CNN
